File: Icarus_FC.kicad_pcb (KiCad board)
At the start: 4 copper layers, 46 x 46 mm, 93 parts, among them IC1 MCP73831T-2ACI_MC, IC2 TXU0304QWBQARQ1, IC3 TLV75518PDRVR, IC4 MAX17048G+T10, J1 JST 1.0mm 6pin GPS, J2 JST 1.0mm 6pin -DJI, J3 Conn_01x20_GPIO, J4 Conn_01x02_MountingPin, J5 Conn_01x04, SW1 SW_RESET, SW2 SW_BOOTSEL, U1 W25Q128JVPIQ, U11 TXU0104BQAR, U13 ICM-20948, U14 ICM-20948, U2 TPS63031DSK, U3 TPS22810DRV, U4 CSNP16GCR01-AOW, U5 RP235x-B, U6 H3LIS200DLTR, U7 BMP390L, U9 ICM-20948, Y1 CM4012M00012001

Commit message: Add files via upload
Parts:
- removed C36: 1uF, Capacitor_SMD:C_0201_0603Metric
- removed C37: 10nF, Capacitor_SMD:C_0402_1005Metric
- removed C38, C39, C40: 0.1uF, Capacitor_SMD:C_0201_0603Metric
- removed IC1: MCP73831T-2ACI_MC, Battery and Power MGMT:SON50P300X200X100-9N-D
- removed IC3: TLV75518PDRVR, Battery and Power MGMT:SON65P200X200X80-7N
- removed IC4: MAX17048G+T10, Battery and Power MGMT:SON50P200X200X80-9N-D
- removed J2: JST 1.0mm 6pin -DJI, Connector_JST:JST_SH_SM06B-SRSS-TB_1x06-1MP_P1.00mm_Horizontal
- removed R2, R31, R32, R33: 10k, Resistor_SMD:R_0201_0603Metric
- removed R3: 2K, Resistor_SMD:R_0201_0603Metric
- removed U13, U14, U9: ICM-20948, Package_DFN_QFN:QFN-24-1EP_3x3mm_P0.4mm_EP1.75x1.6mm
- added C22: 0.1uF, Capacitor_SMD:C_0201_0603Metric, F.Cu at (187.4, 72.7)
- added C25: 0.1uF, Capacitor_SMD:C_0201_0603Metric, F.Cu at (173.4, 81.7)
- added C26: 0.1uF, Capacitor_SMD:C_0201_0603Metric, F.Cu at (170.4, 72.2)
- added D2: LED, LED_SMD:LED_0201_0603Metric, F.Cu at (165.4, 59.2)
- added G***: LOGO, LOGO, F.Cu at (166.8, 79.8)
- added G***: LOGO, LOGO, B.Cu at (185.1, 84.3)
- added G***: LOGO, LOGO, B.Cu at (187.4, 81.6)
- added J6: Conn_01x08_MountingPin, Connector_JST:JST_SH_SM08B-SRSS-TB_1x08-1MP_P1.00mm_Horizontal, B.Cu at (175.0, 93.7)
- added R20: 10k, Resistor_SMD:R_0201_0603Metric, F.Cu at (172.5, 86.4)
- added R21: 10k, Resistor_SMD:R_0201_0603Metric, F.Cu at (179.3, 87.0)
- added R22: 33, Resistor_SMD:R_0201_0603Metric, F.Cu at (187.8, 75.5)
- added R24: 1.2k, Resistor_SMD:R_0201_0603Metric, F.Cu at (175.5, 64.7)
- added R25: 10k, Resistor_SMD:R_0201_0603Metric, F.Cu at (171.4, 62.8)
- added R26: 1.2k, Resistor_SMD:R_0201_0603Metric, F.Cu at (172.5, 63.2)
- added U10: H3LIS100DLTR, H3LIS200DLTR:PQFN50P300X300X100-16N, F.Cu at (177.6, 83.5)
- added U8: BQ24075RGTR, Battery and Power MGMT:QFN50P300X300X100-17N, F.Cu at (173.0, 65.8)
- C1: value 0.1uF -> 10uF; footprint Capacitor_SMD:C_0201_0603Metric -> Capacitor_SMD:C_0402_1005Metric
- C10, C9: value 0.1uF -> 12pF
- C12, C14, C29: value 4.7uF -> 0.1uF
- C16: value 10uF -> 0.1uF; footprint Capacitor_SMD:C_0402_1005Metric -> Capacitor_SMD:C_0201_0603Metric
- C17, C18, C19, C27: value 0.1uF -> 4.7uF
- C23: value 4.7uF -> 10nF
- C24, C32: value 22uF -> 0.1uF; footprint Capacitor_SMD:C_0402_1005Metric -> Capacitor_SMD:C_0201_0603Metric
- C35: value 1uF -> 0.1uF
- C4: value 12pF -> 4.7uF
- C5: value 12pF -> 0.1uF
- C6, C8: value 0.1uF -> 22uF; footprint Capacitor_SMD:C_0201_0603Metric -> Capacitor_SMD:C_0402_1005Metric
- C7: value 0.1uF -> 1uF
- D1: value LED_Small -> LED; footprint LED_SMD:LED_0402_1005Metric -> LED_SMD:LED_0201_0603Metric
- IC2: value TXU0304QWBQARQ1 -> MAX17048G+T10; footprint Battery and Power MGMT:TXU0304QWBQARQ1 -> Battery and Power MGMT:SON50P200X200X80-9N-D
- J1: value JST 1.0mm 6pin GPS -> Conn_01x04; footprint Connector_JST:JST_SH_SM06B-SRSS-TB_1x06-1MP_P1.00mm_Horizontal -> Connector_JST:JST_SH_SM04B-SRSS-TB_1x04-1MP_P1.00mm_Horizontal
- J3: value Conn_01x20_GPIO -> JST 1.0mm 6pin -DJI; footprint Connector_JST:JST_SHL_SM12B-SHLS-TF_1x12-1MP_P1.00mm_Horizontal -> Connector_JST:JST_SH_SM06B-SRSS-TB_1x06-1MP_P1.00mm_Horizontal; moved to F.Cu
- J4: value Conn_01x02_MountingPin -> JST 1.0mm 6pin GPS; footprint Connector_Molex:Molex_PicoBlade_53261-0271_1x02-1MP_P1.25mm_Horizontal -> Connector_JST:JST_SH_SM06B-SRSS-TB_1x06-1MP_P1.00mm_Horizontal; moved to F.Cu
- J5: value Conn_01x04 -> C122410; footprint Connector_JST:JST_SH_SM04B-SRSS-TB_1x04-1MP_P1.00mm_Horizontal -> Connector_Molex:Molex_PicoBlade_53398-0271_1x02-1MP_P1.25mm_Vertical
- L1: value 3.3uH -> 2.2uH; footprint Inductor_SMD:L_Wuerth_MAPI-2512 -> Battery and Power MGMT:ASMPM-0806
- L2: value 2.2uH -> 3.3uH; footprint Battery and Power MGMT:L0806 -> Battery and Power MGMT:ASMPM-0806
- R1: value 10k -> 100K
- R10: value 10k -> 27R
- R11: value 27R -> 100K
- R12: value 10k -> 2K
- R13: value 560K -> 10k
- R14, R4: value 100K -> 10k
- R5: value 470 -> 1K
- R6: value 27R -> 1K
- R7: value 27R -> 10k
- R8: value 100K -> 27R
- R9: value 2K -> 27R
- SW1: value SW_RESET -> SW_BOOTSEL
- SW2: value SW_BOOTSEL -> SW_RESET
- U11: value TXU0104BQAR -> BMP390L; footprint BQA0014A-MFG:BQA0014A-MFG -> BMP:10LGA_2X2X0p75_BOS
- U2: footprint Package_SON:WSON-10-1EP_2.5x2.5mm_P0.5mm_EP1.2x2mm -> Package_SON:WSON-10-1EP_2.5x2.5mm_P0.5mm_EP1.2x2mm_ThermalVias
- U3: value TPS22810DRV -> RP2350-A; footprint Package_SON:WSON-6-1EP_2x2mm_P0.65mm_EP1x1.6mm -> SMD Components:QFN-60-1EP_7x7mm_P0.4mm_EP3.4x3.4mm_ThermalVias
- U4: value CSNP16GCR01-AOW -> TPS22810DRV; footprint Package_LGA:LGA-8_8x6.2mm_P1.27mm -> Package_SON:WSON-6-1EP_2x2mm_P0.65mm_EP1x1.6mm
- U5: value RP235x-B -> CSNP16GCR01-AOW; footprint RP2350B:QFN-80-1EP_10x10mm_P0.4mm_EP3.4x3.4mm_ThermalVias -> Package_LGA:LGA-8_8x6.2mm_P1.27mm
- U6: value H3LIS200DLTR -> MMC5983MA; footprint H3LIS200DLTR:PQFN50P300X300X100-16N -> IMU's:PQFN50P300X300X100-16N
- U7: value BMP390L -> ICM-45686; footprint BMP:10LGA_2X2X0p75_BOS -> ICM_45686:IC_ICM-45686
- moved J1 37.3 mm to (175.0, 56.6), turned to 180 degrees
- moved logoB 37.1 mm to (174.4, 57.0)
- moved R17 36.2 mm to (193.8, 68.4), turned to -90 degrees
- moved J3 33.7 mm to (157.6, 70.1)
- moved logo 33.1 mm to (175.0, 94.7)
- moved R16 32.2 mm to (192.5, 68.4), turned to -90 degrees
- moved R15 28.2 mm to (191.2, 68.4), turned to -90 degrees
- moved J4 27.5 mm to (157.7, 79.9), turned to -90 degrees
- moved C33 26.6 mm to (184.8, 59.0)
- moved C1 25.6 mm to (174.9, 87.9)
- moved C27 23.7 mm to (189.6, 68.1), turned to 0 degrees
- moved C2 23.5 mm to (162.1, 65.7)
- moved R11 23.2 mm to (186.8, 79.8)
- moved QRCode 22.7 mm to (182.1, 62.1)
- moved U1 22.4 mm to (182.1, 62.1)
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- renumbered G*** to QRCode, G*** to icon, G*** to logo, G*** to logoB
Connections:
- C1 pad 1: VBAT -> Net-(U6-CAP)
- C10 pad 1: +3V3 -> Net-(U3-XOUT)
- C12 pad 1: Net-(U5-VREG_AVDD) -> +3V3
- C16 pad 1: +1.1V -> +3V3
- C17 pad 1: +1.1V -> +3V3
- C18 pad 1: +1.1V -> Net-(U3-VREG_AVDD)
- C20 pad 1: GND -> +1.1V
- C20 pad 2: +1V8 -> GND
- C21 pad 1: Net-(U9-REGOUT) -> +1.1V
- C23 pad 1: VBAT -> GND
- C23 pad 2: GND -> Net-(U4-CT)
- C24 pad 1: VBAT -> +3V3
- C27 pad 1: Net-(U13-REGOUT) -> GND
- C27 pad 2: GND -> +3V3
- C28 pad 1: Net-(U14-REGOUT) -> GND
- C28 pad 2: GND -> +3V3
- C29 pad 1: GND -> +3V3
- C29 pad 2: +3V3 -> GND
- C3 pad 1: +5V -> VBATout
- C30 pad 1: +3V3 -> GND
- C30 pad 2: GND -> +3V3
- C31 pad 1: +1V8 -> +3V3
- C33 pad 1: GND -> +3V3
- C33 pad 2: +1V8 -> GND
- C35 pad 1: +1V8 -> GND
- C35 pad 2: GND -> +3V3
- C4 pad 1: Net-(U5-XIN) -> GND
- C4 pad 2: GND -> +5V
- C5 pad 1: Net-(U5-XOUT) -> VBAT
- C6 pad 1: +3V3 -> VBATout
- C7 pad 1: +3V3 -> GND
- C7 pad 2: GND -> +3V3
- C9 pad 1: +3V3 -> Net-(U3-XIN)
- H1 pad 1: (no net) -> GND
- H2 pad 1: (no net) -> GND
- H3 pad 1: (no net) -> GND
- H4 pad 1: (no net) -> GND
- IC2 pad 1: +3V3 -> GND
- IC2 pad 2: /GPIO4 -> VBAT
- IC2 pad 3: /GPIO3 -> VBAT
- IC2 pad 4: /GPIO9 -> GND
- IC2 pad 5: /GPIO2 -> unconnected-(IC2-~{ALRT}-Pad5)
- IC2 pad 6: unconnected-(IC2-NC_1-Pad6) -> GND
- IC2 pad 7: GND -> /GPIO3
- IC2 pad 8: +3V3 -> /GPIO2
- IC2 pad 9: unconnected-(IC2-NC_2-Pad9) -> GND
- J1 pad 1: /GPIO1 -> GND
- J1 pad 2: /GPIO0 -> /USB_D-
- J1 pad 3: GND -> /USB_D+
- J1 pad 4: +3V3 -> +5V
- J1 pad MP: GND -> (no net)
- J3 pad 1: GND -> Net-(J3-Pin_1)
- J3 pad 2: VBAT -> GND
- J3 pad 3: +3V3 -> unconnected-(J3-Pin_3-Pad3)
- J3 pad 4: /GPIO31 -> unconnected-(J3-Pin_4-Pad4)
- J3 pad 5: /GPIO32 -> unconnected-(J3-Pin_5-Pad5)
- J3 pad 6: /GPIO33 -> unconnected-(J3-Pin_6-Pad6)
- J4 pad 1: VBAT -> GND
- J4 pad 2: GND -> +3V3
- J5 pad 1: GND -> VBAT
- J5 pad 2: /USB_D- -> GND
- J5 pad MP: (no net) -> GND
- L1 pad 1: +1.1V -> Net-(U2-L2)
- L1 pad 2: Net-(U5-VREG_XL) -> Net-(U2-L1)
- L2 pad 1: Net-(U2-L2) -> +1.1V
- L2 pad 2: Net-(U2-L1) -> Net-(U3-VREG_LX)
- R1 pad 1: /GPIO31 -> /~{QSPI_CS}
- R10 pad 1: /CS_BMP390L -> +3V3
- R10 pad 2: +3V3 -> Net-(U3-VREG_AVDD)
- R11 pad 2: Net-(U5-VREG_AVDD) -> /~{RESET}
- R12 pad 1: +3V3 -> /BOOTSEL
- R12 pad 2: /GPIO9 -> /~{QSPI_CS}
- R13 pad 2: Net-(U2-FB) -> /GPIO25
- R14 pad 1: Net-(U2-FB) -> +3V3
- R14 pad 2: GND -> /GPIO26
- R15 pad 2: /GPIO25 -> /GPIO24
- R16 pad 2: /GPIO26 -> /GPIO23
- R17 pad 2: /GPIO24 -> /GPIO22
- R18 pad 2: /GPIO23 -> /GPIO8
- R19 pad 2: /GPIO22 -> /GPIO5
- R4 pad 1: /~{QSPI_CS_{0}} -> /GPIO2
- R5 pad 1: Net-(D1-A) -> Net-(D2-A)
- R6 pad 1: /D- -> Net-(D1-A)
- R6 pad 2: /USB_D- -> +5V
- R7 pad 1: /D+ -> /GPIO3
- R7 pad 2: /USB_D+ -> +3V3
- R8 pad 1: +3V3 -> /D-
- R8 pad 2: /~{RESET} -> /USB_D-
- R9 pad 1: /BOOTSEL -> /D+
- R9 pad 2: /~{QSPI_CS_{0}} -> /USB_D+
- U1 pad 1: /~{QSPI_CS_{0}} -> /~{QSPI_CS}
- U11 pad 10: /CS_BMP390L_1.8V -> +3V3
- U11 pad 2: /GPIO7 -> /GPIO14
- U11 pad 3: /GPIO6 -> GND
- U11 pad 4: /GPIO5 -> /GPIO15
- U11 pad 5: /CS_BMP390L -> /GPIO12
- U11 pad 6: unconnected-(U11-NC-Pad6) -> /BMP390L_CS
- U11 pad 7: GND -> unconnected-(U11-INT/DNC-Pad7)
- U11 pad 8: +3V3 -> GND
- U11 pad 9: unconnected-(U11-NC-Pad9) -> GND
- U2 pad 10: Net-(U2-FB) -> +3V3
- U2 pad 5: VBAT -> VBATout
- U2 pad 6: VBAT -> VBATout
- U2 pad 7: GND -> VBATout
- U2 pad 8: VBAT -> VBATout
- U3 pad 1: Net-(J2-Pin_1) -> +3V3
- U3 pad 2: unconnected-(U3-QOD-Pad2) -> /GPIO0
- U3 pad 3: Net-(U3-CT) -> /GPIO1
- U3 pad 4: GND -> /GPIO2
- U3 pad 5: /CAM_CTRL -> /GPIO3
- U3 pad 6: VBAT -> +1.1V
- U3 pad 7: GND -> /GPIO4
- U4 pad 1: /GPIO25 -> Net-(J3-Pin_1)
- U4 pad 2: /GPIO26 -> unconnected-(U4-QOD-Pad2)
- U4 pad 3: /GPIO21 -> Net-(U4-CT)
- U4 pad 5: /GPIO22 -> /CAM_CTRL
- U4 pad 6: /GPIO23 -> VBAT
- U4 pad 7: /GPIO24 -> GND
- U5 pad 1: /GPIO4 -> /GPIO25
- U5 pad 2: /GPIO5 -> /GPIO26
- U5 pad 3: /GPIO6 -> Net-(U5-SCLK)
- U5 pad 4: /GPIO7 -> GND
- U5 pad 5: +3V3 -> /GPIO22
- U5 pad 6: /CS_BMP390L -> /GPIO23
- U5 pad 7: /GPIO9 -> /GPIO24
- U5 pad 8: /GPIO10 -> +3V3
- U6 pad 1: +1V8 -> /GPIO14
- U6 pad 10: GND -> Net-(U6-CAP)
- U6 pad 11: unconnected-(U6-INT_1-Pad11) -> GND
- U6 pad 12: GND -> unconnected-(U6-NC__4-Pad12)
- U6 pad 13: GND -> +3V3
- U6 pad 14: +3V3 -> unconnected-(U6-NC__5-Pad14)
- U6 pad 15: +3V3 -> unconnected-(U6-INT-Pad15)
- U6 pad 16: GND -> /GPIO15
- U6 pad 2: (no net) -> +3V3
- U6 pad 3: (no net) -> unconnected-(U6-NC-Pad3)
- U6 pad 4: /SCK_1.8V -> /GPIO11
- U6 pad 5: GND -> /GPIO12
- U6 pad 6: /MOSI_1.8V -> unconnected-(U6-NC__1-Pad6)
- U6 pad 7: /MISO_1.8V -> unconnected-(U6-NC__2-Pad7)
- U6 pad 8: /HighG_IMU_CS_1.8V -> unconnected-(U6-NC__3-Pad8)
- U6 pad 9: unconnected-(U6-INT_2-Pad9) -> GND
- U7 pad 1: +1V8 -> /GPIO4
- U7 pad 10: +1V8 -> unconnected-(U7-RESV/AUX1_CS-Pad10)
- U7 pad 2: /SCK_1.8V -> unconnected-(U7-RESV/AUX1_SDIO/AUX1_SDI/MAS_DA-Pad2)
- U7 pad 3: GND -> unconnected-(U7-RESV/AUX1_SCLK/MAS_CLK-Pad3)
- U7 pad 4: /MOSI_1.8V -> unconnected-(U7-INT1/INT-Pad4)
- U7 pad 5: /MISO_1.8V -> +3V3
- U7 pad 6: /CS_BMP390L_1.8V -> GND
- U7 pad 8: GND -> +3V3
- U7 pad 9: GND -> unconnected-(U7-INT2/FSYNC/CLKIN-Pad9)
- Y1 pad 1: Net-(U5-XOUT) -> Net-(U3-XOUT)
- Y1 pad 3: Net-(U5-XIN) -> Net-(U3-XIN)
Routing:
- net /GPIO32: track 101.1 -> 0.00 mm, vias 4 -> 0
- net +1V8: track 94.2 -> 0.00 mm, vias 10 -> 0
- net /CS1_1.8V: track 74.4 -> 0.00 mm, vias 4 -> 0
- net +3V3: track 258.7 -> 200.6 mm, vias 11 -> 8
- net /MISO_1.8V: track 55.3 -> 0.00 mm, vias 5 -> 0
- net /MOSI_1.8V: track 52.2 -> 0.00 mm, vias 3 -> 0
- net /SCK_1.8V: track 48.6 -> 0.00 mm, vias 7 -> 0
- net /GPIO31: track 42.7 -> 0.00 mm, vias 2 -> 0
- net /GPIO19: track 0.00 -> 31.8 mm, vias 0 -> 3
- net /HighG_IMU_CS_1.8V: track 30.0 -> 0.00 mm, vias 2 -> 0
- net /GPIO0: track 51.1 -> 23.3 mm, vias 2 -> 0
- net /GPIO17: track 0.00 -> 27.8 mm, vias 0 -> 3
- net /GPIO16: track 0.00 -> 27.4 mm, vias 0 -> 3
- net /GPIO18: track 0.00 -> 26.7 mm, vias 0 -> 3
- net /GPIO14: track 0.00 -> 25.8 mm, vias 0 -> 2
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- added copper zone on F.Cu, net +3V3
- added copper zone on B.Cu, net +5V
- added copper zone on F.Cu, net +5V
- added copper zone on F.Cu, net Net-(J3-Pin_1)
- added copper zone on F.Cu, net VBAT
- added copper zone on F.Cu, net VBATout
Other:
- board text added: "1S lipo/0-100G 16MB Rom/512MB SDIO"
- board text added: "Boot"
- board text added: "CAM"
- board text added: "GND 3V3 RX TX X X"
- board text added: "Rest"
- board text added: "VBAT GND 9 10 16 17 18 19"
- board text added: "X"
- board text added: "Y"
- board text added: "Z"
- board text removed: "39 -> 31 3V3 VBAT GND"
- board text removed: "RX TX GND 3V3 SDA SCL"
