File: Icarus_FC.kicad_sch (KiCad schematic)
At the start: 89 parts, among them IC1 MCP73831T-2ACI_MC, IC2 TXU0304QWBQARQ1, IC3 TLV75518PDRVR, IC4 MAX17048G+T10, J1 JST 1.0mm 6pin GPS, J2 JST 1.0mm 6pin -DJI, J3 Conn_01x20_GPIO, J4 Conn_01x02_MountingPin, J5 Conn_01x04, SW1 SW_RESET, SW2 SW_BOOTSEL, U1 W25Q128JVPIQ, U11 TXU0104BQAR, U13 ICM-20948, U14 ICM-20948, U2 TPS63031DSK, U3 TPS22810DRV, U4 CSNP16GCR01-AOW, U5 RP235x-B, U6 H3LIS200DLTR, U7 BMP390L, U9 ICM-20948, Y1 CM4012M00012001

Commit message: Add files via upload
Parts:
- removed C23: 4.7uF, Capacitor_SMD:C_0201_0603Metric, symbol Device:C_Small
- removed C27, C28, C34, C6, C8: 0.1uF, Capacitor_SMD:C_0201_0603Metric, symbol Device:C_Small
- removed C35, C36: 1uF, Capacitor_SMD:C_0201_0603Metric, symbol Device:C_Small
- removed C5: 12pF, Capacitor_SMD:C_0201_0603Metric, symbol Device:C_Small
- removed D1: LED_Small, LED_SMD:LED_0402_1005Metric, symbol Device:LED_Small
- removed H1, H2, H3, H4: MountingHole, TestPoint:TestPoint_Plated_Hole_D2.0mm, symbol Mechanical:MountingHole
- removed IC1: MCP73831T-2ACI_MC, Battery and Power MGMT:SON50P300X200X100-9N-D, symbol MCP73831T-2ACI_MC:MCP73831T-2ACI_MC
- removed IC2: TXU0304QWBQARQ1, Battery and Power MGMT:TXU0304QWBQARQ1, symbol TXU0304QWBQARQ1:TXU0304QWBQARQ1
- removed IC3: TLV75518PDRVR, Battery and Power MGMT:SON65P200X200X80-7N, symbol TLV75518PDRVR:TLV75518PDRVR
- removed J3: Conn_01x20_GPIO, Connector_JST:JST_SHL_SM12B-SHLS-TF_1x12-1MP_P1.00mm_Horizontal, symbol Connector_Generic_MountingPin:Conn_01x20_MountingPin
- removed R10, R12, R31, R32, R33: 10k, Resistor_SMD:R_0201_0603Metric, symbol Device:R
- removed R13: 560K, Resistor_SMD:R_0201_0603Metric, symbol Device:R_Small
- removed R14: 100K, Resistor_SMD:R_0201_0603Metric, symbol Device:R_Small
- removed R3: 2K, Resistor_SMD:R_0201_0603Metric, symbol Device:R_Small
- removed R7: 27R, Resistor_SMD:R_0201_0603Metric, symbol Device:R_Small
- removed U11: TXU0104BQAR, BQA0014A-MFG:BQA0014A-MFG, symbol 2025-12-15_03-39-19:TXU0104BQAR
- removed U13, U14, U9: ICM-20948, Package_DFN_QFN:QFN-24-1EP_3x3mm_P0.4mm_EP1.75x1.6mm, symbol 00_lcsc:ICM-20948
- removed U5: RP235x-B, RP2350B:QFN-80-1EP_10x10mm_P0.4mm_EP3.4x3.4mm_ThermalVias, symbol MCU_RaspberryPi:RP235x-B
- added C1: 10uF, Capacitor_SMD:C_0402_1005Metric, symbol Device:C_Small
- added C20, C22, C24, C25, C26, C29: 0.1uF, Capacitor_SMD:C_0201_0603Metric, symbol Device:C_Small
- added D1, D2: LED, LED_SMD:LED_0201_0603Metric, symbol Device:LED
- added J6: Conn_01x08_MountingPin, Connector_JST:JST_SH_SM08B-SRSS-TB_1x08-1MP_P1.00mm_Horizontal, symbol Connector_Generic_MountingPin:Conn_01x08_MountingPin
- added R10: 27R, Resistor_SMD:R_0201_0603Metric, symbol Device:R_Small
- added R12: 2K, Resistor_SMD:R_0201_0603Metric, symbol Device:R_Small
- added R18, R19, R20, R21, R25: 10k, Resistor_SMD:R_0201_0603Metric, symbol Device:R
- added R22: 33, Resistor_SMD:R_0201_0603Metric, symbol Device:R
- added R24, R26: 1.2k, Resistor_SMD:R_0201_0603Metric, symbol Device:R
- added U3: RP2350-A, SMD Components:QFN-60-1EP_7x7mm_P0.4mm_EP3.4x3.4mm_ThermalVias, symbol MCU_RaspberryPi:RP235x-A
- added U6: MMC5983MA, IMU's:PQFN50P300X300X100-16N, symbol MMC5983MA:MMC5983MA
- added U7: ICM-45686, ICM_45686:IC_ICM-45686, symbol ICM-45686:ICM-45686
- added U8: BQ24075RGTR, Battery and Power MGMT:QFN50P300X300X100-17N, symbol BQ24075RGTR:BQ24075RGTR
- C10, C9: value 0.1uF -> 12pF
- C12, C14: value 4.7uF -> 0.1uF
- C16: value 10uF -> 0.1uF; footprint Capacitor_SMD:C_0402_1005Metric -> Capacitor_SMD:C_0201_0603Metric
- C17, C18, C19: value 0.1uF -> 4.7uF
- C23: renamed from C37; footprint Capacitor_SMD:C_0402_1005Metric -> Capacitor_SMD:C_0201_0603Metric
- C4: value 12pF -> 4.7uF
- C7: value 0.1uF -> 1uF
- J5: renamed from J4; value Conn_01x02_MountingPin -> C122410; footprint Connector_Molex:Molex_PicoBlade_53261-0271_1x02-1MP_P1.25mm_Horizontal -> Connector_Molex:Molex_PicoBlade_53398-0271_1x02-1MP_P1.25mm_Vertical
- L1: value 3.3uH -> 2.2uH; footprint Inductor_SMD:L_Wuerth_MAPI-2512 -> Battery and Power MGMT:ASMPM-0806; LCSC C5832359 -> C17701149
- L2: value 2.2uH -> 3.3uH; footprint Battery and Power MGMT:L0806 -> Battery and Power MGMT:ASMPM-0806; LCSC C695610 -> C42411119
- R11: value 27R -> 100K
- R5: value 470 -> 1K
- R6: value 27R -> 1K
- R8: value 100K -> 27R
- R9: value 2K -> 27R
- U10: renamed from U6; value H3LIS200DLTR -> H3LIS100DLTR
- U2: footprint Package_SON:WSON-10-1EP_2.5x2.5mm_P0.5mm_EP1.2x2mm -> Package_SON:WSON-10-1EP_2.5x2.5mm_P0.5mm_EP1.2x2mm_ThermalVias
- renumbered C29 to C27, C38 to C28, C40 to C32, C39 to C34, C20 to C35, C1 to C5, C24 to C6, C32 to C8, IC4 to IC2, J5 to J1, J2 to J3, J1 to J4, R4 to R1, R15 to R13, R16 to R14, R17 to R15, R18 to R16, R19 to R17, R1 to R4, R2 to R7, SW2 to SW1, SW1 to SW2, U7 to U11, U3 to U4, U4 to U5
Connections:
- net HighG_IMU_CS_1.8V is gone; now on net GPIO5: U10.8 (CS)
- net +1.1V: now also C21.1, L2.1, C20.1, C22.1, U3.23 (DVDD), U3.39 (DVDD), U3.50 (VREG_FB), U3.6 (DVDD); no longer C16.1, C17.1, C18.1, L1.1
- net +3V3: now also C12.1, C16.1, C17.1, C30.2, C31.1, C32.1, C33.1, C35.2, C7.2, J4.2 (Pin_2), U10.1 (VDD_IO), U11.1 (VDDIO), U11.10 (VDD), U2.10 (FB), C24.1, C25.2, C29.1, R10.1, R18.1, R19.1, R20.1, R21.1, U3.1 (IOVDD), U3.11 (IOVDD), U3.20 (IOVDD), U3.30 (IOVDD), U3.38 (IOVDD), U3.44 (IOVDD), U3.45 (IOVDD), U3.49 (VREG_VIN), U3.53 (IOVDD), U3.54 (IOVDD), U6.13 (VDDIO), U6.2 (VDD), U7.5 (VDDIO), U7.8 (VDD); no longer C10.1, C30.1, C7.1, C9.1, J4.4 (Pin_4), R8.1
- net +5V: now also C4.2, R6.2, U8.13 (IN), U8.5 (EN2); no longer C3.1
- net BOOTSEL: now also SW2.1 (A), R12.1; no longer R9.1, SW1.1 (A)
- net CAM_CTRL: now also U3.42 (GPIO28)
- net D+: now also R9.1, U3.52 (USB_D+)
- net D-: now also R8.1, U3.51 (USB_D-); no longer R6.1
- net GND: now also C30.1, C33.2, C4.1, C7.1, J4.1 (Pin_1), SW1.1 (A), SW2.2 (B), C1.2, C20.2, C22.2, C24.2, C25.1, C26.2, C29.2, J6.2 (Pin_2), J6.MP (MountPin), R24.1, R25.2, R26.1, U3.47 (GND), U3.61 (GND), U6.11 (GND__1), U6.9 (GND), U7.6 (GND), U8.15 (SYSOFF), U8.17 (EXP), U8.4 (~{CE}), U8.6 (EN1), U8.8 (VSS); no longer C30.2, C33.1, C4.2, C7.2, J4.3 (Pin_3), SW1.2 (B), SW2.1 (A), U2.7 (PS/SYNC)
- net GPIO0: now also J4.4 (Pin_4), U3.2 (GPIO0); no longer J4.2 (Pin_2)
- net GPIO1: now also J4.3 (Pin_3), U3.3 (GPIO1); no longer J4.1 (Pin_1)
- net GPIO10: now also J6.4 (Pin_4), U3.14 (GPIO10)
- net GPIO11: now also R21.2, U3.15 (GPIO11), U6.4 (~{SPI_CS})
- net GPIO12: now also U11.5 (SDO/DNC/SA0), U3.16 (GPIO12), U6.5 (SPI_SDO)
- net GPIO14: now also U11.2 (SCK/SCL), U3.18 (GPIO14), U6.1 (SCL/SPI_SCK)
- net GPIO15: now also U11.4 (SDI/SDO/SDA), U3.19 (GPIO15), U6.16 (SDA/SPI_SDI)
- net GPIO16: now also J6.5 (Pin_5), U3.27 (GPIO16)
- net GPIO17: now also J6.6 (Pin_6), U3.28 (GPIO17)
- net GPIO18: now also J6.7 (Pin_7), U3.29 (GPIO18)
- net GPIO19: now also J6.8 (Pin_8), U3.31 (GPIO19)
- net GPIO2: now also IC2.8 (SDA), R4.1, U3.4 (GPIO2)
- net GPIO20: now also U3.32 (GPIO20)
- net GPIO21: now also R22.1, U3.33 (GPIO21); no longer U5.3 (SCLK)
- net GPIO22: now also U3.34 (GPIO22)
- net GPIO23: now also U3.35 (GPIO23)
- net GPIO24: now also U3.36 (GPIO24)
- net GPIO25: now also U3.37 (GPIO25)
- net GPIO26: now also U3.40 (GPIO26)
- net GPIO29: now also U3.43 (GPIO29)
- net GPIO3: now also IC2.7 (SCL), R7.1, U3.5 (GPIO3)
- net GPIO4: now also U10.7 (SDO/SA0), U3.7 (GPIO4), U7.1 (AP_SDO/AP_AD0)
- net GPIO5: now also R19.2, U3.8 (GPIO5)
- net GPIO6: now also U10.4 (SCL/SPC), U3.9 (GPIO6), U7.13 (AP_SCL/AP_SCLK)
- net GPIO7: now also U10.6 (SDA/SDI/SDO), U3.10 (GPIO7), U7.14 (AP_SDA/AP_SDIO/AP_SDI)
- net GPIO9: now also J6.3 (Pin_3), U3.13 (GPIO9)
- net QSPI_SCLK: now also U3.56 (QSPI_SCLK)
- net QSPI_SD0: now also U3.57 (QSPI_SD0)
- net QSPI_SD1: now also U3.59 (QSPI_SD1)
- net QSPI_SD2: now also U3.58 (QSPI_SD2)
- net QSPI_SD3: now also U3.55 (QSPI_SD3)
- net SWCLK: now also U3.24 (SWCLK)
- net SWDIO: now also U3.25 (SWDIO)
- net USB_D+: now also R9.2
- net USB_D-: now also R8.2; no longer R6.2
- net VBAT: now also J6.1 (Pin_1), U8.2 (BAT_2), U8.3 (BAT_3); no longer C6.1, U2.5 (VIN), U2.6 (EN), U2.8 (VINA)
- net ~{RESET}: now also R11.2, SW1.2 (B), U3.26 (RUN); no longer R8.2, SW2.2 (B)
- net at U2.2 (L2): now also L1.1; no longer L2.1
- net at U2.4 (L1): now also L1.2; no longer L2.2
- net at R5.1: now also D2.2 (A)
- net at Y1.3: now also C9.1, U3.21 (XIN); no longer C4.1
- net at Y1.1: now also C10.1, U3.22 (XOUT)
- removed net +1V8: C31.1, C32.1, C33.2, C35.2, U10.1 (VDD_IO), U11.1 (VDDIO), U11.10 (VDD)
- net CS_BMP390L_1.8V renamed BMP390L_CS
- net BMP390L_CS: now also R20.2, U3.17 (GPIO13)
- removed net GPIO31: IC2.8 (SDA), J4.5 (Pin_5), R4.1
- removed net GPIO32: IC2.7 (SCL), J4.6 (Pin_6), R7.1
- removed net MISO_1.8V: U10.7 (SDO/SA0), U11.5 (SDO/DNC/SA0)
- removed net MOSI_1.8V: U10.6 (SDA/SDI/SDO), U11.4 (SDI/SDO/SDA)
- removed net SCK_1.8V: U10.4 (SCL/SPC), U11.2 (SCK/SCL)
- net ~{QSPI_CS_{0}} renamed ~{QSPI_CS}
- net ~{QSPI_CS}: now also R12.2, U3.60 (~{QSPI_CS}); no longer R9.2
- new net: R26.2, U8.16 (ISET)
- new net: R25.1, U8.1 (TS)
- new net: C18.1, R10.2, U3.46 (VREG_AVDD)
- new net: R22.2, U5.3 (SCLK)
- new net: C1.1, U6.10 (CAP)
- new net: D1.2 (A), R6.1
- new net: D2.1 (K), U8.7 (~{PGOOD})
- new net: R24.2, U8.12 (ILIM)
- new net: D1.1 (K), U8.9 (~{CHG})
- new net: L2.2, U3.48 (VREG_LX)
- new net GPIO27: U3.41 (GPIO27)
- new net GPIO8: R18.2, U3.12 (GPIO8), U7.12 (AP_CS)
- new net VBATout: C26.1, C3.1, C6.1, U2.5 (VIN), U2.6 (EN), U2.7 (PS/SYNC), U2.8 (VINA), U8.10 (OUT_10), U8.11 (OUT_11)
- no-connect marks 48 -> 18
Other:
- note added: "11"
- note added: "23"
- note added: "30"
- note added: "38"
- note added: "39"
- note added: "44"
- note added: "53"
- note removed: "10"
- note removed: "15"
- note removed: "24"
- note removed: "32"
- note removed: "41"
- note removed: "50"
- note removed: "59"
- note removed: "68"
- note removed: "76"
- moved on the sheet: C2, C23, C27, C28, C32, C34, C35, C5, C6, C8, IC2, J1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
